File: RGB LED Driver.sch (EAGLE design)
At the start: 11 parts, among them IC1 SN74LS244N, J1 691311400105, J2 691311400102, J3 691311400105

Commit message: Periodic updates
Fixed OTA in TwinkleFox and Pacifica
Parts:
- removed R1: 4116R-1-331LF, Bourns_4116R-1-331LF:4116R-1-331LF
- added 8X330R: (no value), resistor-bourns:2NBS16-8
- added USB_POWER: (no value), pinhead:PINHD-1X2
Connections:
- new net N$13: J2.2, USB_POWER.2
- net +5V: now also USB_POWER.1; no longer J2.2
- net N$1: now also 8X330R.12; no longer R1.4
- net N$10: now also 8X330R.5; no longer R1.13
- net N$11: now also 8X330R.15; no longer R1.7
- net N$12: now also 8X330R.16; no longer R1.8
- net N$15: now also 8X330R.4; no longer R1.12
- net N$16: now also 8X330R.3; no longer R1.11
- net N$19: now also 8X330R.2; no longer R1.10
- net N$2: now also 8X330R.11; no longer R1.3
- net N$20: now also 8X330R.1; no longer R1.9
- net N$3: now also 8X330R.10; no longer R1.2
- net N$4: now also 8X330R.9; no longer R1.1
- net N$5: now also 8X330R.8; no longer R1.16
- net N$6: now also 8X330R.7; no longer R1.15
- net N$7: now also 8X330R.6; no longer R1.14
- net N$8: now also 8X330R.14; no longer R1.6
- net N$9: now also 8X330R.13; no longer R1.5
Other:
- moved on the sheet: J2
