File: pcb/Rotary Encoder.brd (EAGLE design)
At the start: 83.5 x 43.2 mm, 7 parts

Commit message: Mid-project updates
Parts:
- added MGT1, MGT2, MGT3, MGT4: BEAGLEBONEBLACK_MOUNTING_HOLE, BeagleBone_Black_Wireless:BEAGLEBONEBLACK_MOUNTING_HOLE
Connections:
- net GND: now also MGT1.P$1, MGT2.P$1, MGT3.P$1, MGT4.P$1
Routing:
- net GND: track 105.2 -> 169.9 mm
- net D3: track 100.9 -> 86.8 mm
- net D1: track 87.4 -> 78.0 mm
- net SDA: track 35.0 -> 38.7 mm
- net VCC: track 105.3 -> 104.7 mm

Commit message: Reassign D1, D2
Connections:
- new net D0: S1.A, W1.JP1.3
- net D1: now also U$1.3; no longer S1.A
- net SCL: no longer U$1.3
Routing:
- net D1: track 78.0 -> 0.00 mm
- net SCL: track 47.8 -> 8.25 mm
- net SDA: track 38.7 -> 6.35 mm
Changed lines of the file:
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@@
 <drawing>
 <settings>
-<setting alwaysvectorfont="yes"/>
+<setting alwaysvectorfont="no"/>
 <setting verticaltext="up"/>
 </settings>
@@
 <wire x1="33.02" y1="39.37" x2="33.02" y2="13.97" width="0.1524" layer="16"/>
 </signal>
-<signal name="D1">
-<contactref element="S1" pad="A"/>
-<contactref element="W1" pad="JP2.3"/>
-<wire x1="66.04" y1="34.925" x2="67.945" y2="33.02" width="0.1524" layer="1"/>
-<wire x1="16.51" y1="34.925" x2="66.04" y2="34.925" width="0.1524" layer="1"/>
-<wire x1="7.62" y1="26.035" x2="16.51" y2="34.925" width="0.1524" layer="1"/>
-<wire x1="7.62" y1="16.51" x2="7.62" y2="26.035" width="0.1524" layer="1"/>
-<wire x1="3.937" y1="16.51" x2="7.62" y2="16.51" width="0.1524" layer="1"/>
-</signal>
 <signal name="D4">
 <contactref element="W1" pad="JP2.6"/>
@@
 <signal name="SCL">
 <contactref element="W1" pad="JP1.4"/>
-<contactref element="U$1" pad="3"/>
-<wire x1="63.5" y1="11.43" x2="35.56" y2="39.37" width="0.1524" layer="16"/>
 <wire x1="70.485" y1="11.43" x2="63.5" y2="11.43" width="0.1524" layer="16"/>
 <wire x1="70.485" y1="10.16" x2="70.485" y2="11.43" width="0.1524" layer="16"/>
@@
 <signal name="SDA">
 <contactref element="W1" pad="JP2.4"/>
+<wire x1="70.485" y1="33.02" x2="70.485" y2="39.37" width="0.1524" layer="16"/>
 <contactref element="U$1" pad="4"/>
-<wire x1="70.485" y1="39.37" x2="38.1" y2="39.37" width="0.1524" layer="16"/>
-<wire x1="70.485" y1="33.02" x2="70.485" y2="39.37" width="0.1524" layer="16"/>
+<wire x1="38.1" y1="39.37" x2="70.485" y2="39.37" width="0" layer="19" extent="16-16"/>
+</signal>
+<signal name="D0">
+<contactref element="S1" pad="A"/>
+<contactref element="W1" pad="JP1.3"/>
+<wire x1="3.937" y1="16.51" x2="67.945" y2="10.16" width="0" layer="19" extent="1-1"/>
+</signal>
+<signal name="D1">
+<contactref element="W1" pad="JP2.3"/>
+<contactref element="U$1" pad="3"/>
+<wire x1="35.56" y1="39.37" x2="67.945" y2="33.02" width="0" layer="19" extent="1-1"/>
 </signal>
 </signals>
